File: AK75.sch (KiCad schematic (older format))
At the start: 194 parts, among them J1 JST_01x04, J2 JST_01x04, J3 JST_01x04, SW1 SW_Push, U1 ATmega32U4-AU, Y1 Resonator_Small

Commit message: assigned footprints for components
Parts:
- D17, D34, D51: renamed from D?; footprint (none) -> random-keyboard-parts:D_SOD-123-Pretty
- MX1, MX10, MX11, MX12, MX13, MX14, MX15, MX16, MX2, MX3, MX4, MX5, MX6, MX7, MX8, MX9: footprint (none) -> MX_Only:MXOnly-1U-NoLED
- MX17, MX34, MX51, MX88: renamed from MX?; footprint (none) -> MX_Only:MXOnly-1U-NoLED
- MX18: renamed from MX17; footprint (none) -> MX_Only:MXOnly-1U-NoLED
- MX19: renamed from MX18; footprint (none) -> MX_Only:MXOnly-1U-NoLED
- MX20: renamed from MX19; footprint (none) -> MX_Only:MXOnly-1U-NoLED
- MX21: renamed from MX20; footprint (none) -> MX_Only:MXOnly-1U-NoLED
- MX22: renamed from MX21; footprint (none) -> MX_Only:MXOnly-1U-NoLED
- MX23: renamed from MX22; footprint (none) -> MX_Only:MXOnly-1U-NoLED
- MX24: renamed from MX23; footprint (none) -> MX_Only:MXOnly-1U-NoLED
- MX25: renamed from MX24; footprint (none) -> MX_Only:MXOnly-1U-NoLED
- MX26: renamed from MX25; footprint (none) -> MX_Only:MXOnly-1U-NoLED
- MX27: renamed from MX26; footprint (none) -> MX_Only:MXOnly-1U-NoLED
- MX28: renamed from MX27; footprint (none) -> MX_Only:MXOnly-1U-NoLED
- MX29: renamed from MX28; footprint (none) -> MX_Only:MXOnly-1U-NoLED
- MX30: renamed from MX29; footprint (none) -> MX_Only:MXOnly-1U-NoLED
- MX31: renamed from MX30; footprint (none) -> MX_Only:MXOnly-2U-NoLED
- MX32: renamed from MX31; footprint (none) -> MX_Only:MXOnly-1U-NoLED
- MX33: renamed from MX32; footprint (none) -> MX_Only:MXOnly-1U-NoLED
- MX35: renamed from MX33; footprint (none) -> MX_Only:MXOnly-1.5U-NoLED
- MX36: renamed from MX34; footprint (none) -> MX_Only:MXOnly-1U-NoLED
- MX37: renamed from MX35; footprint (none) -> MX_Only:MXOnly-1U-NoLED
- MX38: renamed from MX36; footprint (none) -> MX_Only:MXOnly-1U-NoLED
- MX39: renamed from MX37; footprint (none) -> MX_Only:MXOnly-1U-NoLED
- MX40: renamed from MX38; footprint (none) -> MX_Only:MXOnly-1U-NoLED
- MX41: renamed from MX39; footprint (none) -> MX_Only:MXOnly-1U-NoLED
- MX42: renamed from MX40; footprint (none) -> MX_Only:MXOnly-1U-NoLED
- MX43: renamed from MX41; footprint (none) -> MX_Only:MXOnly-1U-NoLED
- MX44: renamed from MX42; footprint (none) -> MX_Only:MXOnly-1U-NoLED
- MX45: renamed from MX43; footprint (none) -> MX_Only:MXOnly-1U-NoLED
- MX46: renamed from MX44; footprint (none) -> MX_Only:MXOnly-1U-NoLED
- MX47: renamed from MX45; footprint (none) -> MX_Only:MXOnly-1U-NoLED
- MX48: renamed from MX46; footprint (none) -> MX_Only:MXOnly-1.5U-NoLED
- MX49: renamed from MX47; footprint (none) -> MX_Only:MXOnly-1U-NoLED
- MX50: renamed from MX48; footprint (none) -> MX_Only:MXOnly-1U-NoLED
- MX52: renamed from MX49; footprint (none) -> MX_Only:MXOnly-1.75U-NoLED
- MX53: renamed from MX50; footprint (none) -> MX_Only:MXOnly-1U-NoLED
- MX54: renamed from MX51; footprint (none) -> MX_Only:MXOnly-1U-NoLED
- MX55: renamed from MX52; footprint (none) -> MX_Only:MXOnly-1U-NoLED
- MX56: renamed from MX53; footprint (none) -> MX_Only:MXOnly-1U-NoLED
- MX57: renamed from MX54; footprint (none) -> MX_Only:MXOnly-1U-NoLED
- MX58: renamed from MX55; footprint (none) -> MX_Only:MXOnly-1U-NoLED
- MX59: renamed from MX56; footprint (none) -> MX_Only:MXOnly-1U-NoLED
- MX60: renamed from MX57; footprint (none) -> MX_Only:MXOnly-1U-NoLED
- MX61: renamed from MX58; footprint (none) -> MX_Only:MXOnly-1U-NoLED
- MX62: renamed from MX59; footprint (none) -> MX_Only:MXOnly-1U-NoLED
- MX63: renamed from MX60; footprint (none) -> MX_Only:MXOnly-1U-NoLED
- MX64: renamed from MX61; footprint (none) -> MX_Only:MXOnly-2.25U-NoLED
- MX65: renamed from MX62; footprint (none) -> MX_Only:MXOnly-2.25U-NoLED
- MX66: renamed from MX63; footprint (none) -> MX_Only:MXOnly-1U-NoLED
- MX67: renamed from MX64; footprint (none) -> MX_Only:MXOnly-1U-NoLED
- MX68: renamed from MX65; footprint (none) -> MX_Only:MXOnly-1U-NoLED
- MX69: renamed from MX66; footprint (none) -> MX_Only:MXOnly-1U-NoLED
- MX70: renamed from MX67; footprint (none) -> MX_Only:MXOnly-1U-NoLED
- MX71: renamed from MX68; footprint (none) -> MX_Only:MXOnly-1U-NoLED
- MX72: renamed from MX69; footprint (none) -> MX_Only:MXOnly-1U-NoLED
- MX73: renamed from MX70; footprint (none) -> MX_Only:MXOnly-1U-NoLED
- MX74: renamed from MX71; footprint (none) -> MX_Only:MXOnly-1U-NoLED
- MX75: renamed from MX72; footprint (none) -> MX_Only:MXOnly-1U-NoLED
- MX76: renamed from MX73; footprint (none) -> MX_Only:MXOnly-2.75U-NoLED
- MX77: renamed from MX74; footprint (none) -> MX_Only:MXOnly-1U-NoLED
- MX78: renamed from MX75; footprint (none) -> MX_Only:MXOnly-1.25U-NoLED
- MX79: renamed from MX76; footprint (none) -> MX_Only:MXOnly-1.25U-NoLED
- MX80: renamed from MX77; footprint (none) -> MX_Only:MXOnly-1.25U-NoLED
- MX81: renamed from MX78; footprint (none) -> MX_Only:MXOnly-6.25U-ReversedStabilizers-NoLED
- MX82: renamed from MX79; footprint (none) -> MX_Only:MXOnly-1.25U-NoLED
- MX83: renamed from MX80; footprint (none) -> MX_Only:MXOnly-1.25U-NoLED
- MX84: renamed from MX81; footprint (none) -> MX_Only:MXOnly-1.25U-NoLED
- MX85: renamed from MX82; footprint (none) -> MX_Only:MXOnly-1.25U-NoLED
- MX86: renamed from MX83; footprint (none) -> MX_Only:MXOnly-1U-NoLED
- MX87: renamed from MX84; footprint (none) -> MX_Only:MXOnly-1U-NoLED
- gave numbers to parts that had none: 1
- renumbered D17 to D18, D18 to D19, D19 to D20, D20 to D21, D21 to D22, D22 to D23, D23 to D24, D24 to D25, D25 to D26, D26 to D27, D27 to D28, D28 to D29, D29 to D30, D30 to D31, D31 to D32, D32 to D33, D33 to D35, D34 to D36, D35 to D37, D36 to D38, D37 to D39, D38 to D40, D39 to D41, D40 to D42, D41 to D43, D42 to D44, D43 to D45, D44 to D46, D45 to D47, D46 to D48, D47 to D49, D48 to D50, D49 to D52, D50 to D53, D51 to D54, D52 to D55, D53 to D56, D54 to D57, D55 to D58, D56 to D59, D57 to D60, D58 to D61, D59 to D62, D60 to D63, D61 to D64, D62 to D65, D63 to D66, D64 to D67, D65 to D68, D66 to D69, D67 to D70, D68 to D71, D69 to D72, D70 to D73, D71 to D74, D72 to D75, D73 to D76, D74 to D77, D75 to D78, D76 to D79, D77 to D80, D78 to D81, D79 to D82, D80 to D83, D81 to D84, D82 to D85, D83 to D86, D84 to D87
