File: AK75.kicad_pcb (KiCad board)
At the start: 2 copper layers, 194 parts, among them J1 JST_01x04, J2 JST_01x04, J3 JST_01x04, SW1 SW_Push, U1 ATmega32U4-AU, Y1 Resonator_Small

Commit message: sorted components
Parts:
- C1, C2, C3, C4, C5, D1, D10, D11, D12, D13, D14, D15, D16, D17, D18, D19, D2, D20, D21, D22, D23, D24, D25, D26, D27, D28, D29, D3, D30, D31, D32, D33, D34, D35, D36, D37, D38, D39, D4, D40, D41, D42, D43, D44, D45, D46, D47, D48, D49, D5, D50, D51, D52, D53, D54, D55, D56, D57, D58, D59, D6, D60, D61, D62, D63, D64, D65, D66, D67, D68, D69, D7, D70, D71, D72, D73, D74, D75, D76, D77, D78, D79, D8, D80, D81, D82, D83, D84, D85, D86, D87, D88, D9, J1, J2, J3, R1, R2, R3, R4, R5, R6, R7, U1, Y1: moved to B.Cu
- moved D11 431.3 mm to (138.6, 209.0)
- moved D20 431.3 mm to (121.4, 209.0)
- moved D23 431.3 mm to (132.9, 209.0)
- moved D28 431.3 mm to (127.1, 209.0)
- moved D34 431.3 mm to (115.6, 209.0)
- moved D10 431.1 mm to (132.9, 205.6)
- moved D13 431.1 mm to (121.4, 205.6)
- moved D25 431.1 mm to (127.1, 205.6)
- moved D32 431.1 mm to (115.6, 205.6)
- moved D9 431.1 mm to (138.6, 205.6)
- moved D31 407.2 mm to (159.1, 183.3)
- moved D37 407.2 mm to (153.4, 183.3)
- moved D42 397.6 mm to (123.5, 172.6)
- moved D33 395.3 mm to (123.5, 176.0)
- moved D21 393.1 mm to (129.2, 179.3)
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
Commit message: initial diode placement
Parts:
- moved D34 285.7 mm to (361.9, 64.3)
- moved D51 279.3 mm to (361.9, 83.3)
- moved D17 268.3 mm to (361.9, 40.5)
- moved D15 254.8 mm to (323.9, 40.5)
- moved D32 251.7 mm to (323.9, 64.3)
- moved D16 250.8 mm to (342.9, 40.5)
- moved D33 246.2 mm to (342.9, 64.3)
- moved D49 241.4 mm to (323.9, 83.3)
- moved D14 241.3 mm to (300.0, 40.5)
- moved D88 229.5 mm to (361.9, 140.5)
- moved D77 228.9 mm to (342.9, 121.4)
- moved D13 226.4 mm to (276.2, 40.5)
- moved D86 216.9 mm to (323.9, 140.5)
- moved D50 211.9 mm to (342.9, 83.3)
- moved D12 211.8 mm to (257.2, 40.5)
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